Commit message: right arm, safeguards and ik fixes

File: urdf/nico_left_arm.urdf (robot description, URDF)
Before this commit: robot complete, 8 links, 7 joints
Joints:
- joint l_wrist_z: origin xyz=0 -0.010201 -0.14055 rpy=3.141593 0 0.028703 -> xyz=0 -0.010201 -0.11055 rpy=3.141593 0 0.028703

File: urdf/nico_right_arm.urdf (robot description, URDF)
Before this commit: robot complete, 17 links, 16 joints
Joints:
- joint r_wrist_z: origin xyz=0 0.0102 -0.14105 rpy=0 0 0.028946 -> xyz=0 0.0102 -0.11105 rpy=0 0 0.028946
