Commit message: implicit coordinate transfer net

File: urdf/nico_right_arm.urdf (robot description, URDF)
Before this commit: robot complete, 17 links, 16 joints
Links:
- removed link finger_segment:11
- removed link finger_segment:12
- removed link finger_segment:13
- removed link finger_segment:21
- removed link finger_segment:22
- removed link finger_segment:23
- removed link fingertip:11
- removed link fingertip:12
- removed link fingertip:13
Joints:
- removed joint r_indexfinger_1st_x
- removed joint r_indexfinger_2nd_x
- removed joint r_indexfingers_x
- removed joint r_ringfinger_1st_x
- removed joint r_ringfinger_2nd_x
- removed joint r_ringfingers_x
- removed joint r_thumb_1st_x
- removed joint r_thumb_2nd_x
- removed joint r_thumb_x
